File: pathfinder.kicad_pcb (KiCad board)
At the start: 2 copper layers, 90.9 x 76.6 mm, 20 parts, among them SW1 SW_Push, SW2 SW_Push, SW3 SW_Push, SW4 SW_Push, SW5 SW_Push, SW6 SW_Push, U1 XIAO-RP2040-DIP, U2 OLED_0.91_128x32

Commit message: fix
Parts:
- added REF**: MountingHole_3.2mm_M3, MountingHole:MountingHole_3.2mm_M3, F.Cu at (116.5, 71.9)
- added REF**: MountingHole_3.2mm_M3, MountingHole:MountingHole_3.2mm_M3, F.Cu at (192.7, 86.2)
- added REF**: MountingHole_3.2mm_M3, MountingHole:MountingHole_3.2mm_M3, F.Cu at (116.5, 86.2)
- added REF**: MountingHole_3.2mm_M3, MountingHole:MountingHole_3.2mm_M3, F.Cu at (192.7, 71.9)
- D10, D11, D12, D7, D8, D9: footprint SK6812 Mini-E:SK6812MINI-E_fixed -> footprints:SK6812MINI-E_fixed
- U1: footprint XIAO RP SERIES:XIAO-RP2040-DIP -> Hackclub Footprints:XIAO-RP2040-DIP
Routing:
- net GND: track 36.9 -> 67.4 mm, vias 11 -> 15
- net COL3: track 76.1 -> 74.7 mm
- net COL2: track 77.7 -> 77.8 mm, vias 1 -> 3
Other:
- board text added: "吃好睡好活好学好(≧◡≦)"
- board text removed: "电路也有心跳 (≧◡≦)<3"
