File: _autosave-pathfinder.kicad_pcb (KiCad board)
At the start: 2 copper layers, 67.1 x 69.1 mm, 20 parts, among them SW1 SW_Push, SW2 SW_Push, SW3 SW_Push, SW4 SW_Push, SW5 SW_Push, SW6 SW_Push, U1 XIAO-RP2040-DIP, U2 OLED_0.91_128x32

Commit message: fix
Parts:
- added REF**: MountingHole_3.2mm_M3, MountingHole:MountingHole_3.2mm_M3, F.Cu at (116.5, 69.5)
- added REF**: MountingHole_3.2mm_M3, MountingHole:MountingHole_3.2mm_M3, F.Cu at (195.1, 69.5)
- added REF**: MountingHole_3.2mm_M3, MountingHole:MountingHole_3.2mm_M3, F.Cu at (166.5, 117.2)
- added REF**: MountingHole_3.2mm_M3, MountingHole:MountingHole_3.2mm_M3, F.Cu at (145.1, 117.2)
Connections:
- U1 pad 7: ENC_A -> unconnected-(U1-GPIO0/TX-Pad7)
- U1 pad 8: ENC_B -> unconnected-(U1-GPIO1/RX-Pad8)_1
- U1 pad 9: ENC_SW -> unconnected-(U1-GPIO2/SCK-Pad9)_1
Routing:
- net ROW2: track 115.3 -> 111.4 mm
- net ENC_SW: track 1.08 -> 0.00 mm
- net (no net): track 0.00 -> 1.08 mm
Other:
- board size 67.1 x 69.1 mm -> 90.9 x 76.6 mm
- board text added: "好好学习，天天向上"
- board text added: "电路也有心跳 (≧◡≦)<3"
