File: pathfinder.kicad_sch (KiCad schematic)
At the start: 29 parts, among them SW1 SW_Push, SW2 SW_Push, SW3 SW_Push, SW4 SW_Push, SW5 SW_Push, SW6 SW_Push, SW7 SW_Push, SW8 SW_Push, SW9 SW_Push, U1 XIAO-RP2040-DIP, U2 OLED_0.91_128x32

Commit message: fix
Parts:
- removed D13, D14, D15, D16, D17, D18: SK6812MINI-E, Hackclub Footprints:MX_SK6812MINI-E_REV, symbol Hackclub Symbols:SK6812MINI-E
- removed D7, D8, D9: D, Diode_THT:D_DO-35_SOD27_P7.62mm_Horizontal, symbol Device:D
- removed SW7, SW8, SW9: SW_Push, Button_Switch_Keyboard:SW_Cherry_MX_1.00u_PCB, symbol Switch:SW_Push
- added D7, D8, D9: SK6812MINI-E, Hackclub Footprints:MX_SK6812MINI-E_REV, symbol Hackclub Symbols:SK6812MINI-E
- added SW7: RotaryEncoder_Switch, Rotary_Encoder:RotaryEncoder_Alps_EC11E-Switch_Vertical_H20mm, symbol Device:RotaryEncoder_Switch
Connections:
- net ROW3 is gone; now on net COL2: U1.3 (GPIO28/ADC2/A2)
- net COL2: no longer U1.9 (GPIO2/SCK)
- net GND: now also D7.3 (VSS), D8.3 (VSS), D9.3 (VSS), SW7.C, SW7.S1
- net at U1.11 (GPIO3/MOSI): now also D7.4 (DIN)
- net ENC_B: now reaches U1.8 (GPIO1/RX)
- net ENC_B: now also SW7.B
- net DIN1: no longer names the net of D10.4 (DIN)
- net DIN1: now also D9.2 (DOUT); no longer U1.7 (GPIO0/TX)
- net VBUS renamed 5V
- net 5V: now also D7.1 (VDD), D8.1 (VDD), D9.1 (VDD)
- new net: D8.2 (DOUT), D9.4 (DIN)
- new net: D7.2 (DOUT), D8.4 (DIN)
- new net ENC_A: SW7.A, U1.7 (GPIO0/TX)
- new net ENC_SW: SW7.S2, U1.9 (GPIO2/SCK)
- no-connect marks 3 -> 1
Other:
- moved on the sheet: U2

Commit message: fix
Parts:
- removed SW7: RotaryEncoder_Switch, Rotary_Encoder:RotaryEncoder_Alps_EC11E-Switch_Vertical_H20mm, symbol Device:RotaryEncoder_Switch
Connections:
- net ENC_A: no longer names the net of U1.7 (GPIO0/TX)
- net ENC_B: no longer names the net of U1.8 (GPIO1/RX)
- net ENC_SW: no longer names the net of U1.9 (GPIO2/SCK)
- no-connect marks 1 -> 4
