File: pathfinder.kicad_sch (KiCad schematic)
At the start: 20 parts, among them SW1 SW_Push, SW2 SW_Push, SW3 SW_Push, SW4 SW_Push, SW5 SW_Push, SW6 SW_Push, U1 XIAO-RP2040-DIP, U2 OLED_0.91_128x32

Commit message: fix
Parts:
- D10, D11, D12, D7, D8, D9: footprint SK6812 Mini-E:SK6812MINI-E_fixed -> footprints:SK6812MINI-E_fixed
- U1: footprint XIAO RP SERIES:XIAO-RP2040-DIP -> Hackclub Footprints:XIAO-RP2040-DIP
Changed lines of the file:
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@@
 			)
 		)
-		(property "Footprint" "SK6812 Mini-E:SK6812MINI-E_fixed"
+		(property "Footprint" "footprints:SK6812MINI-E_fixed"
 			(at 185.42 67.31 0)
 			(effects
@@
 			)
 		)
-		(property "Footprint" "SK6812 Mini-E:SK6812MINI-E_fixed"
+		(property "Footprint" "footprints:SK6812MINI-E_fixed"
 			(at 246.38 67.31 0)
 			(effects
@@
 			)
 		)
-		(property "Footprint" "SK6812 Mini-E:SK6812MINI-E_fixed"
+		(property "Footprint" "footprints:SK6812MINI-E_fixed"
 			(at 200.66 67.31 0)
 			(effects
@@
 			)
 		)
-		(property "Footprint" "XIAO RP SERIES:XIAO-RP2040-DIP"
+		(property "Footprint" "Hackclub Footprints:XIAO-RP2040-DIP"
 			(at 93.218 76.708 0)
 			(effects
@@
 			)
 		)
-		(property "Footprint" "SK6812 Mini-E:SK6812MINI-E_fixed"
+		(property "Footprint" "footprints:SK6812MINI-E_fixed"
 			(at 170.18 67.31 0)
 			(effects
@@
 			)
 		)
-		(property "Footprint" "SK6812 Mini-E:SK6812MINI-E_fixed"
+		(property "Footprint" "footprints:SK6812MINI-E_fixed"
 			(at 215.9 67.31 0)
 			(effects
@@
 			)
 		)
-		(property "Footprint" "SK6812 Mini-E:SK6812MINI-E_fixed"
+		(property "Footprint" "footprints:SK6812MINI-E_fixed"
 			(at 231.14 67.31 0)
 			(effects
